File: board schematics (EAGLE)/droneHAT.brd (EAGLE design)
At the start: 65 x 56 mm, 37 parts, among them IC1 V_REG_MIC2920, IC2 5V, IC3 ACS712, J1 XBEE-1B1, J2 BAT, J3 ADAFRUITIMU, J4 ADAFRUITGPS, J5 BAT, K1 PIN20X2, M1 SMALL_SERVO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

Commit message: Updated Board
Parts:
- added D4, D5, D6, D7: GREEN, SparkFun-LED:LED-1206
- added M4: SMALL_SERVO, SparkFun-Electromechanical:1X03
- added R6, R7, R8, R9: 1k, adafruit:M1206
- IC2: device SparkFun-PowerIC:TO220-IGO -> SparkFun-PowerIC:TSRN1
- moved C13 2.10 mm to (55.6, 14.6), turned to 0 degrees
- moved C12 2.01 mm to (61.6, 12.7)
- moved IC2 1.90 mm to (59.0, 19.1)
- moved C11 1.42 mm to (50.8, 20.3), turned to 45 degrees
- moved C5 1.27 mm to (16.5, 10.8)
- moved R5 0.63 mm to (55.6, 11.2)
Connections:
- removed net RXD0: D2.A, R2.2, U1.2
- removed net TXD0: K1.8, U1.3
- removed net XB-CTS: J1.12, U1.82
- new net N$10: D6.C, R8.2
- new net N$11: D7.A, R9.2
- new net N$2: M1.2, M2.2, M3.2, M4.2
- new net N$4: D4.A, J1.6
- new net N$5: D4.C, R6.1
- new net N$6: D5.C, R7.2
- new net RPI-RXD0: D2.A, R2.2, U1.3
- new net RPI-TXD0: K1.8, U1.2
- new net SERV4: M4.1, U1.23
- net +5V: now also IC2.3, R9.1; no longer IC2.OUT, M1.2, M2.2, M3.2
- net GND: now also IC2.2, M4.3, R6.2, R7.1, R8.1; no longer IC2.GND
- net GRDY: now also D5.A
- net LIN1: now also D6.A
- net LRDY: now also D7.C
- net SERV1: now also U1.41; no longer U1.25
- net SERV2: now also U1.25; no longer U1.24
- net SERV3: now also U1.24; no longer U1.23
- net VIN: now also IC2.1; no longer IC2.IN
Routing:
- net XB-CTS: track 37.4 -> 0.00 mm
- net TXD0: track 25.9 -> 0.00 mm
- net RPI-TXD0: track 0.00 -> 23.2 mm
- net +5V: track 255.0 -> 271.3 mm
- net RPI-RXD0: track 0.00 -> 15.4 mm
- net GRDY: track 52.9 -> 68.2 mm
- net LIN1: track 18.4 -> 33.6 mm
- net SERV1: track 18.1 -> 32.9 mm
- net RXD0: track 13.7 -> 0.00 mm
- net SERV4: track 0.00 -> 13.1 mm
- net GND: track 133.2 -> 143.7 mm, vias 6 -> 7
- net N$4: track 0.00 -> 10.5 mm
- net N$10: track 0.00 -> 8.98 mm
- net N$2: track 0.00 -> 7.62 mm
- net LRDY: track 20.2 -> 25.2 mm
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