File: board schematics (EAGLE)/droneHAT.sch (EAGLE design)
At the start: 37 parts, among them IC1 V_REG_MIC2920, IC2 5V, IC3 ACS712, J1 XBEE-1B1, J2 BAT, J3 ADAFRUITIMU, J4 ADAFRUITGPS, J5 BAT, K1 PIN20X2, M1 SMALL_SERVO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

Commit message: Updated Board
Parts:
- added D4, D5, D6, D7: GREEN, SparkFun-LED:LED-GREENLARGE
- added M4: SMALL_SERVO, SparkFun-Electromechanical:SMALL_SERVO
- added R6, R7, R8, R9: 1k, adafruit:R-US_M1206
- IC2: device SparkFun-PowerIC:V_REG_78XXSINK -> SparkFun-PowerIC:V_REG_78XX
Connections:
- removed net RXD0: D2.A, R2.2, U1.(RXD0/PCIN8)PE0
- removed net TXD0: K1.8, U1.(TXD0)PE1
- removed net XB-CTS: J1.CTS, U1.PK7(ADC15/PCINT23)
- new net N$10: D6.C, R8.2
- new net N$11: D7.A, R9.2
- new net N$2: M1.V+, M2.V+, M3.V+, M4.V+
- new net N$4: D4.A, J1.RSSI
- new net N$5: D4.C, R6.1
- new net N$6: D5.C, R7.2
- new net RPI-RXD0: D2.A, R2.2, U1.(TXD0)PE1
- new net RPI-TXD0: K1.8, U1.(RXD0/PCIN8)PE0
- new net SERV4: M4.SIG, U1.(OC2A/PCINT4)PB4
- net +5V: now also R9.1; no longer M1.V+, M2.V+, M3.V+
- net GND: now also M4.GND, R6.2, R7.1, R8.1
- net GRDY: now also D5.A
- net LIN1: now also D6.A
- net LRDY: now also D7.C
- net SERV1: now also U1.PL6; no longer U1.(OC1B/PCINT6)PB6
- net SERV2: now also U1.(OC1B/PCINT6)PB6; no longer U1.(OC1A/PCINT5)PB5
- net SERV3: now also U1.(OC1A/PCINT5)PB5; no longer U1.(OC2A/PCINT4)PB4
Other:
- moved on the sheet: J3, JP1
